File: schematic/guitar_interface/mcu.kicad_sch (KiCad schematic)
At the start: 35 parts, among them J1 Conn_ST_STDC14, U8 STM32F446VETx, Y1 LFXTAL032878

Commit message: fix minor issues and do most of the pcb layout
Connections:
- net 3.3V is gone; now on net VPP_3.3V: J1.3 (VCC), R46.2
Changed lines of the file:
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@@
+	)
+	(junction
+		(at 107.95 20.32)
+		(diameter 0)
+		(color 0 0 0 0)
 	)
 	(junction
@@
 	)
 	(junction
+		(at 120.65 20.32)
+		(diameter 0)
+		(color 0 0 0 0)
+	)
+	(junction
 		(at 40.64 20.32)
 		(diameter 0)
@@
 	(wire
 		(pts
+			(xy 107.95 20.32) (xy 120.65 20.32)
+		)
+		(stroke
+			(width 0)
+			(type default)
+		)
+	)
+	(wire
+		(pts
 			(xy 151.13 39.37) (xy 151.13 35.56)
 		)
@@
 	(wire
 		(pts
+			(xy 54.61 34.29) (xy 107.95 34.29)
+		)
+		(stroke
+			(width 0)
+			(type default)
+		)
+	)
+	(wire
+		(pts
 			(xy 71.12 20.32) (xy 85.09 20.32)
 		)
@@
 	(wire
 		(pts
+			(xy 107.95 34.29) (xy 107.95 20.32)
+		)
+		(stroke
+			(width 0)
+			(type default)
+		)
+	)
+	(wire
+		(pts
 			(xy 146.05 181.61) (xy 146.05 184.15)
 		)
@@
 	(wire
 		(pts
+			(xy 120.65 20.32) (xy 120.65 34.29)
+		)
+		(stroke
+			(width 0)
+			(type default)
+		)
+	)
+	(wire
+		(pts
 			(xy 171.45 77.47) (xy 233.68 77.47)
 		)
@@
 	(wire
 		(pts
+			(xy 54.61 93.98) (xy 54.61 34.29)
+		)
+		(stroke
+			(width 0)
+			(type default)
+		)
+	)
+	(wire
+		(pts
 			(xy 85.09 27.94) (xy 90.17 27.94)
 		)
@@
 	(wire
 		(pts
-			(xy 104.14 20.32) (xy 143.51 20.32)
-		)
-		(stroke
-			(width 0)
-			(type default)
-		)
-	)
-	(wire
-		(pts
-			(xy 120.65 31.75) (xy 120.65 34.29)
+			(xy 104.14 20.32) (xy 107.95 20.32)
 		)
 		(stroke
@@
 	(wire
 		(pts
+			(xy 41.91 93.98) (xy 54.61 93.98)
+		)
+		(stroke
+			(width 0)
+			(type default)
+		)
+	)
+	(wire
+		(pts
 			(xy 30.48 36.83) (xy 43.18 36.83)
 		)
@@
 	(wire
 		(pts
+			(xy 120.65 20.32) (xy 143.51 20.32)
+		)
+		(stroke
+			(width 0)
+			(type default)
+		)
+	)
+	(wire
+		(pts
 			(xy 187.96 95.25) (xy 195.58 95.25)
 		)
@@
 			(width 0)
 			(type default)
-		)
-	)
-	(label "3.3V"
-		(at 120.65 31.75 0)
-		(effects
-			(font
-				(size 1.27 1.27)
-			)
-			(justify left bottom)
 		)
 	)
@@
 		(effects
 			(font
-				(size 1.27 1.27)
-			)
-			(justify left bottom)
-		)
-	)
-	(label "3.3V"
-		(at 41.91 93.98 0)
-		(effects
-			(font
