File: schematic/guitar_interface/guitar_interface.kicad_sch (KiCad schematic)
At the start: 9 parts, among them J2 MUSBRM1C1M06, J3 Conn_01x02_Pin, J4 Conn_01x02_Pin

Commit message: refine layout fix, fix some minor issues, add additional ground planes on all layers, and add mounting holes
Parts:
- J3, J4: footprint Connector_PinSocket_1.00mm:PinSocket_1x02_P1.00mm_Vertical -> Connector_PinSocket_2.54mm:PinSocket_1x02_P2.54mm_Vertical
Changed lines of the file:
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@@
 			)
 		)
-		(property "Footprint" "Connector_PinSocket_1.00mm:PinSocket_1x02_P1.00mm_Vertical"
+		(property "Footprint" "Connector_PinSocket_2.54mm:PinSocket_1x02_P2.54mm_Vertical"
 			(at 222.25 90.17 0)
 			(effects
@@
 			)
 		)
-		(property "Footprint" "Connector_PinSocket_1.00mm:PinSocket_1x02_P1.00mm_Vertical"
+		(property "Footprint" "Connector_PinSocket_2.54mm:PinSocket_1x02_P2.54mm_Vertical"
 			(at 33.02 95.25 0)
 			(effects
